File: uBITz Platform Code/Host/Schem/uBITz-Host-Reference-Impl/05-6309-Based-Host/uBITz-Host-6309-Host/uBITz-Host-6309-Host.kicad_sch (KiCad schematic)
At the start: 24 parts, among them J3 Conn_01x02_Pin, J4 Conn_02x05_Top_Bottom, U1 MC6809E, U11 24LC16BT-I_SN, U5 ATF1504AS-10AU100, Y1 ACH-14.31818MHZ-EK

Commit message: Corrected for bus width (20 -> 19) and allowd mapper to rewrite bits A13-A15 of the address bus (become PA13-PA15)
Connections:
- net A13: no longer J1.B34 (A13)
- net A14: no longer J1.B37 (A14)
- net A15: no longer J1.B38 (A15)
- net PA14: now reaches U5.75 (I/O)
- net PA14: now also J1.B37 (A14)
- net PA15: now reaches U5.79 (I/O)
- net PA15: now also J1.B38 (A15)
- net A16 renamed PA16
- net A17 renamed PA17
- net A18 renamed PA18
- net A19: no longer names the net of J1.B46 (A19)
- net A19: no longer U5.35 (I/O)
- new net PA13: J1.B34 (A13), U5.35 (I/O)
- no-connect marks 70 -> 69

Commit message: Beautify board and schematic Added PDF
Other:
- note added: "Allows for JTAG Recovery Add jumper to send 12V to CPLD during programming to recover JTAG pins"
- note added: "Dual Diodes to power the CPLD only from JTAB OR from the +5V from the backplane This is to allow programming the CPLD from JTAG without powering the rest of the Host board"
- note added: "GND bank from Edge connector"
- note added: "Memory Mapper and Bus adaptor. Use ATF1504-10AU100 or ATF1508-10AU100"
- note added: "We don't support multiple CPUs so LIC, AVMA and TSC are NC"
- note removed: "Dual Diodes to power the CPLD only from USB OR from the +5V from the backplane This is to allow programming the CPLD from USB without powering the rest of the Host board"
- moved on the sheet: J1B, J1C
