File: uBITz Platform Code/Host/Schem/uBITz-Host-Reference-Impl/03-Z80-Based-Host/uBITz-Host-z80-Host/uBITz-Host-z80-Host.kicad_sch (KiCad schematic)
At the start: 44 parts, among them J1 Conn_01x02_Pin, J2 12401610E4_2A, U1 Z084000xP, U2 MAX662ACSA_T, U3 24LC16BT-I_SN, U4 SN74LS612N, U5 ATF1504AS-10AU100, U6 FT232H, U7 93LC56BT-I/OT, Y1 ACH-14.31818MHZ-EK, Y2 ECS-2033-120-BN

Commit message: Removed the Serial Profile and first commit of the a Host
Parts:
- added J3: ~, Connector_PCBEdge:BUS_PCIexpress_x16, symbol Host:CORE_CONNECTOR
Connections:
- net +5V: now also J3.A2 (+5V_MAIN), J3.A3 (+5V_MAIN), J3.B1 (+5V_MAIN), J3.B2 (+5V_MAIN), J3.B3 (+5V_MAIN)
- net A0: now also J3.B14 (A0)
- net A1: now also U5.8 (I/O), J3.B15 (A1); no longer U5.7 (NC)
- net A10: now also J3.B31 (A10)
- net A11: now also J3.B33 (A11)
- net A12: now also J3.B34 (A12)
- net A13: now also J3.B37 (A13)
- net A14: now also J3.B38 (A14)
- net A15: now also J3.B41 (A15)
- net A16: now also J3.B42 (A16)
- net A17: now also J3.B45 (A17)
- net A18: now also J3.B46 (A18)
- net A19: now also J3.B48 (A19)
- net A2: now also U5.9 (I/O), J3.B17 (A2); no longer U5.8 (I/O)
- net A20: now also J3.B50 (A20)
- net A21: now also J3.B51 (A21)
- net A22: now also J3.B54 (A22)
- net A23: now also J3.B55 (A23)
- net A3: now also U5.10 (I/O), J3.B19 (A3); no longer U5.9 (I/O)
- net A4: now also U5.12 (I/O/PD1), J3.B20 (A4); no longer U5.10 (I/O)
- net A5: now also U5.13 (I/O), J3.B23 (A5); no longer U5.12 (I/O/PD1)
- net A6: now also U5.14 (I/O), J3.B24 (A6); no longer U5.13 (I/O)
- net A7: now also U5.16 (I/O), J3.B27 (A7); no longer U5.14 (I/O)
- net A8: now also J3.B28 (A8)
- net A9: now also J3.B30 (A9)
- net BUS_R/~{W}: now also J3.A11 (R/~{W})
- net BUS_SCL: now also J3.B5 (SLOT_SCL)
- net BUS_SDA: now also J3.B6 (SLOT_SDA)
- net B_D10: now also U5.75 (I/O)
- net D0: now also J3.A16 (D0)
- net D1: now also J3.A17 (D1)
- net D2: now also J3.A19 (D2)
- net D3: now also J3.A21 (D3)
- net D4: now also J3.A22 (D4)
- net D5: now also J3.A25 (D5)
- net D6: now also J3.A26 (D6)
- net D7: now also J3.A29 (D7)
- net GND: now also J3.A12 (GND), J3.A15 (GND), J3.A18 (GND), J3.A23 (GND), J3.A24 (GND), J3.A27 (GND), J3.A28 (GND), J3.A30 (D8), J3.A31 (GND), J3.A32 (D9), J3.A33 (D10), J3.A34 (GND), J3.A35 (D11), J3.A36 (D12), J3.A37 (GND), J3.A38 (GND), J3.A39 (D13), J3.A4 (GND), J3.A40 (D14), J3.A41 (GND), J3.A42 (GND), J3.A43 (D15), J3.A44 (D16), J3.A45 (GND), J3.A46 (GND), J3.A47 (D17), J3.A48 (D18), J3.A49 (GND), J3.A50 (D19), J3.A51 (GND), J3.A52 (D20), J3.A53 (D21), J3.A54 (GND), J3.A55 (GND), J3.A56 (D22), J3.A57 (D23), J3.A58 (GND), J3.A59 (GND), J3.A60 (D24), J3.A61 (D25), J3.A62 (GND), J3.A63 (GND), J3.A64 (D26), J3.A65 (D27), J3.A66 (GND), J3.A67 (GND), J3.A68 (D28), J3.A69 (D29), J3.A70 (GND), J3.A71 (GND), J3.A72 (D30), J3.A73 (D31), J3.A74 (GND), J3.A75 (GND), J3.A78 (GND), J3.A79 (GND), J3.A82 (GND), J3.B13 (GND), J3.B16 (GND), J3.B21 (GND), J3.B22 (GND), J3.B25 (GND), J3.B26 (GND), J3.B29 (GND), J3.B32 (GND), J3.B35 (GND), J3.B36 (GND), J3.B39 (GND), J3.B4 (GND), J3.B40 (GND), J3.B43 (GND), J3.B44 (GND), J3.B47 (GND), J3.B49 (GND), J3.B52 (GND), J3.B53 (GND), J3.B56 (GND), J3.B57 (GND), J3.B58 (A24), J3.B59 (A25), J3.B60 (GND), J3.B61 (GND), J3.B62 (A26), J3.B63 (A27), J3.B64 (GND), J3.B65 (GND), J3.B66 (A28), J3.B67 (A29), J3.B68 (GND), J3.B69 (GND), J3.B7 (GND), J3.B70 (A30), J3.B71 (A31), J3.B72 (GND), J3.B73 (GND), J3.B76 (GND), J3.B77 (GND), J3.B80 (GND)
- net ~{BUS_CPU_ACK}: now also J3.B11 (~{CPU_ACK})
- net ~{BUS_CPU_INT}: now also J3.A77 (~{CPU_INT0}), J3.A80 (~{CPU_INT1}), J3.B79 (~{CPU_INT2}), J3.B81 (~{CPU_INT3})
- net ~{BUS_CPU_NMI}: now also J3.A81 (~{CPU_NMI0}), J3.B82 (~{CPU_NMI1})
- net ~{BUS_IORQ}: now also J3.A6 (~{IORQ})
- net ~{BUS_READY}: now also J3.A76 (~{READY})
- net ~{BUS_RESET}: now also J3.A5 (~{RESET})
- net ~{M1}: now also U5.41 (I/O); no longer U5.16 (I/O)
- no-connect marks 30 -> 47

Commit message: Committing the first fully completed version of the Z80 based host
Parts:
- removed unit 2 of J3
- added C19, C20, C21, C22, C23, C24, C29, C30: 100n, Capacitor_SMD:C_0603_1608Metric_Pad1.08x0.95mm_HandSolder, symbol Device:C
- added unit 2 of J1
- added J4: Conn_02x05_Top_Bottom, Connector_PinHeader_2.54mm:PinHeader_2x05_P2.54mm_Vertical, symbol Connector_Generic:Conn_02x05_Top_Bottom
- added U10, U12, U13, U6, U8, U9: SN74LVC245ADGVR, Footprints:DGV20-M, symbol Host:SN74LVC245ADGVR
- C17: renamed from C21; value 100n -> 10u
- C18: renamed from C22; value 100n -> 10u
- R6: renamed from R1; footprint (none) -> Resistor_SMD:R_0603_1608Metric_Pad0.98x0.95mm_HandSolder
- U3: renamed from U6; value FT232H -> FT232HL; footprint (none) -> Footprints:QFP50P900X900X160-48N
- U4: renamed from U7; footprint Footprints:SOT-23-6_MC_MCH-L -> SOT-23-6_MC_MCH
- U5: footprint Footprints:100A_ATM-L -> Footprints:100A_ATM
- renumbered C6 to C1, C16 to C10, C17 to C11, C18 to C12, C19 to C13, C20 to C14, C10 to C15, C11 to C16, C5 to C2, C4 to C25, C2 to C26, C1 to C27, C3 to C28, C7 to C3, C8 to C4, C9 to C5, C12 to C6, C13 to C7, C14 to C8, C15 to C9, J3 to J1, J1 to J3, R6 to R1, R4 to R2, R5 to R3, R7 to R4, R8 to R5, R3 to R7, R2 to R8, U4 to U1, U3 to U11, U1 to U2, U2 to U7
Connections:
- net B_~{MM} is gone; now on net MAP_~{MM}: U1.13 (~{MM})
- net +12V: now also J4.1 (Pin_1)
- net +5V: now also C29.1, C30.1; no longer U2.25 (~{BUSREQ})
- net +5V_CPLD: now also J4.2 (Pin_2)
- net A0: now also U5.16 (I/O), U6.9 (A8); no longer J1.B14 (A0), U5.6 (I/O)
- net A1: now also U5.14 (I/O), U6.8 (A7); no longer J1.B15 (A1), U5.8 (I/O)
- net A10: now also U8.7 (A6); no longer J1.B31 (A10)
- net A11: now also U8.6 (A5); no longer J1.B33 (A11)
- net A12: now also U8.5 (A4); no longer J1.B34 (A12)
- net A13: now also U8.4 (A3); no longer J1.B37 (A13)
- net A14: now also U8.3 (A2); no longer J1.B38 (A14)
- net A15: now also U8.2 (A1); no longer J1.B41 (A15)
- net A16: now also U9.9 (A8); no longer J1.B42 (A16)
- net A17: now also U9.8 (A7); no longer J1.B45 (A17)
- net A18: now also U9.7 (A6); no longer J1.B46 (A18)
- net A19: now also U9.6 (A5); no longer J1.B48 (A19)
- net A2: now also U5.13 (I/O), U6.7 (A6); no longer J1.B17 (A2), U5.9 (I/O)
- net A20: now also U9.5 (A4); no longer J1.B50 (A20)
- net A21: now also U9.4 (A3); no longer J1.B51 (A21)
- net A22: now also U9.3 (A2); no longer J1.B54 (A22)
- net A23: now also U9.2 (A1); no longer J1.B55 (A23)
- net A3: now also U5.12 (I/O/PD1), U6.6 (A5); no longer J1.B19 (A3), U5.10 (I/O)
- net A4: now also U5.10 (I/O), U6.5 (A4); no longer J1.B20 (A4), U5.12 (I/O/PD1)
- net A5: now also U5.9 (I/O), U6.4 (A3); no longer J1.B23 (A5), U5.13 (I/O)
- net A6: now also U5.8 (I/O), U6.3 (A2); no longer J1.B24 (A6), U5.14 (I/O)
- net A7: now also U5.6 (I/O), U6.2 (A1); no longer J1.B27 (A7), U5.16 (I/O)
- net A8: now also U8.9 (A8); no longer J1.B28 (A8)
- net A9: now also U8.8 (A7); no longer J1.B30 (A9)
- net BUS_R/~{W}: now also U12.1 (DIR), U13.4 (A3); no longer J1.A11 (R/~{W})
- net CPUCLK: now also U13.9 (A8)
- net D0: now also U12.2 (A1); no longer J1.A16 (D0)
- net D1: now also U12.3 (A2); no longer J1.A17 (D1)
- net D2: now also U12.4 (A3); no longer J1.A19 (D2)
- net D3: now also U12.5 (A4); no longer J1.A21 (D3)
- net D4: now also U12.6 (A5); no longer J1.A22 (D4)
- net D5: now also U12.7 (A6); no longer J1.A25 (D5)
- net D6: now also U12.8 (A7); no longer J1.A26 (D6)
- net D7: now also U12.9 (A8); no longer J1.A29 (D7)
- net GND: now also C19.2, C20.2, C21.2, C22.2, C23.2, C24.2, C29.2, C30.2, J1.A12 (GND), J1.A15 (GND), J1.A18 (GND), J1.A23 (GND), J1.A24 (GND), J1.A27 (GND), J1.A28 (GND), J1.A30 (GND), J1.A34 (GND), J1.A37 (GND), J1.A38 (GND), J1.A4 (GND), J1.A41 (GND), J1.A42 (GND), J1.A45 (GND), J1.A46 (GND), J1.A5 (GND), J1.A50 (GND), J1.A51 (GND), J1.A54 (GND), J1.A55 (GND), J1.A58 (GND), J1.A59 (GND), J1.A6 (GND), J1.A62 (GND), J1.A63 (GND), J1.A66 (GND), J1.A67 (GND), J1.A70 (GND), J1.A71 (GND), J1.A73 (GND), J1.B11 (GND), J1.B13 (GND), J1.B16 (GND), J1.B21 (GND), J1.B22 (GND), J1.B25 (GND), J1.B26 (GND), J1.B29 (GND), J1.B32 (GND), J1.B35 (GND), J1.B36 (GND), J1.B39 (GND), J1.B4 (GND), J1.B40 (GND), J1.B43 (GND), J1.B44 (GND), J1.B47 (GND), J1.B48 (GND), J1.B52 (GND), J1.B53 (GND), J1.B56 (GND), J1.B57 (GND), J1.B60 (GND), J1.B61 (GND), J1.B64 (GND), J1.B65 (GND), J1.B68 (GND), J1.B69 (GND), J1.B7 (GND), J1.B8 (GND), J4.10 (Pin_10), U10.10 (GND), U10.2 (A1), U10.3 (A2), U10.4 (A3), U10.5 (A4), U10.6 (A5), U10.7 (A6), U10.8 (A7), U10.9 (A8), U12.10 (GND), U13.10 (GND), U6.10 (GND), U8.10 (GND), U9.10 (GND); no longer J1.A30 (D8), J1.A32 (D9), J1.A33 (D10), J1.A35 (D11), J1.A36 (D12), J1.A39 (D13), J1.A40 (D14), J1.A43 (D15), J1.A44 (D16), J1.A47 (D17), J1.A48 (D18), J1.A50 (D19), J1.A52 (D20), J1.A53 (D21), J1.A56 (D22), J1.A57 (D23), J1.A60 (D24), J1.A61 (D25), J1.A64 (D26), J1.A65 (D27), J1.A68 (D28), J1.A69 (D29), J1.A72 (D30), J1.A73 (D31), J1.B58 (A24), J1.B59 (A25), J1.B62 (A26), J1.B63 (A27), J1.B66 (A28), J1.B67 (A29), J1.B70 (A30), J1.B71 (A31), J3.2 (Pin_2), R1.2, U1.21 (~{ME}), U5.32 (I/O), U5.52 (I/O), U5.54 (I/O), U5.56 (I/O), U5.57 (I/O), U5.58 (I/O), U5.60 (I/O), U5.61 (I/O), U5.63 (I/O), U5.64 (I/O), U5.65 (I/O), U5.67 (I/O), U5.68 (I/O), U5.69 (I/O), U5.88 (INPUT/OE1)
- net TCK: now also J4.6 (Pin_6)
- net TDI: now also J4.7 (Pin_7)
- net TDO: now also J4.8 (Pin_8)
- net TMS: now also J4.9 (Pin_9)
- net VCCD: now also R1.2, U3.12 (VCCIO), U3.46 (VCCIO)
- net ~{BUS_CPU_ACK}: now also U13.2 (A1); no longer J1.B11 (~{CPU_ACK})
- net ~{BUS_CPU_INT}: now also J1.A76 (~{CPU_INT0}), J1.A78 (~{CPU_INT2}), J1.A79 (~{CPU_INT3}); no longer J1.A80 (~{CPU_INT1}), J1.B79 (~{CPU_INT2}), J1.B81 (~{CPU_INT3})
- net ~{BUS_CPU_NMI}: now also J1.A82 (~{CPU_NMI1}); no longer J1.B82 (~{CPU_NMI1})
- net ~{BUS_IORQ}: now also U13.3 (A2); no longer J1.A6 (~{IORQ})
- net ~{BUS_READY}: now also J1.B79 (~{READY}); no longer J1.A76 (~{READY})
- net ~{BUS_RESET}: now also J1.B73 (~{RESET}), U5.89 (INPUT/GCLR); no longer J1.A5 (~{RESET}), U5.96 (I/O)
- net ~{INT}: now also U5.42 (I/O/PD2); no longer U5.23 (I/O)
- net ~{IORQ}: now also U5.20 (I/O); no longer U5.19 (I/O)
- net ~{M1}: now also U5.33 (I/O); no longer U5.41 (I/O)
- net ~{MREQ}: now also U5.19 (I/O); no longer U5.17 (I/O)
- net ~{NMI}: now also U5.17 (I/O); no longer U5.25 (I/O)
- net ~{RD}: now also U5.23 (I/O); no longer U5.20 (I/O)
- net ~{RESET}: now also U5.32 (I/O); no longer U5.30 (I/O)
- net ~{WAIT}: now also U5.30 (I/O); no longer U5.29 (I/O)
- net B_CLK_HOST: now reaches J1.A7 (CLK_HOST)
- net B_CLK_HOST: now also U13.11 (B8)
- net B_A3: now reaches J1.B18 (A3)
- net B_A3: now also U6.14 (B5)
- net ~{B_MREQ}: now reaches J1.B74 (~{MREQ})
- net ~{B_MREQ}: now also U13.13 (B6)
- net ~{B_MEM0_CS}: now reaches J1.B75 (~{MEM0_CS})
- net ~{B_MEM0_CS}: now also U13.14 (B5)
- net ~{B_IORQ}: now reaches J1.B78 (~{IORQ})
- net ~{B_IORQ}: now also U13.17 (B2)
- net ~{BUSACK}: now reaches U2.23 (~{BUSACK})
- net ~{BUSACK}: now also U5.29 (I/O)
- net +3V3: now reaches J1.A10 (+3V3_MAIN)
- net +3V3: now also J1.A9 (+3V3_MAIN), J1.B10 (+3V3_MAIN), J1.B9 (+3V3_MAIN), C19.1, C20.1, C21.1, C22.1, C23.1, C24.1, U10.1 (DIR), U10.20 (VCC), U12.20 (VCC), U13.1 (DIR), U13.20 (VCC), U6.1 (DIR), U6.20 (VCC), U8.1 (DIR), U8.20 (VCC), U9.1 (DIR), U9.20 (VCC)
- net MAP_~{ME}: now reaches U5.44 (I/O)
- net MAP_~{ME}: now also U1.21 (~{ME})
- net MAP_~{MM}: now reaches U5.45 (I/O)
- net MAP_~{STROBE}: now reaches U5.46 (I/O)
- net MAP_~{STROBE}: now also U1.5 (~{STROBE})
- net MAP_D8: now reaches U5.47 (I/O)
- net MAP_D8: now also U1.31 (D8)
- net MAP_D9: now reaches U5.48 (I/O)
- net MAP_D9: now also U1.32 (D9)
- net B_D10: no longer names the net of U5.75 (I/O)
- net B_D10: no longer U1.33 (D10)
- net B_D11: no longer names the net of U5.71 (I/O)
- net B_D11: no longer U1.34 (D11)
- net B_D8: no longer names the net of U5.79 (I/O)
- net B_D8: no longer U1.31 (D8)
- net B_D9: no longer names the net of U5.76 (I/O)
- net B_D9: no longer U1.32 (D9)
- net B_RS0 renamed MAP_RS0
- net B_RS1 renamed MAP_RS1
- net MAP_RS1: now also U5.40 (I/O); no longer U5.36 (I/O)
- net B_RS2 renamed MAP_RS2
- net B_RS3 renamed MAP_RS3
- net MAP_RS3: now also U5.36 (I/O); no longer U5.40 (I/O)
- net B_~{CS} renamed MAP_~{CS}
- net MAP_~{CS}: now also U5.41 (I/O); no longer U5.31 (I/O)
- removed net B_~{STROBE}: U1.5 (~{STROBE}), U5.33 (I/O)
- net DM renamed D-
- net DP renamed D+
- new net B_A0: J1.B14 (A0), U6.11 (B8)
- new net B_A1: J1.B15 (A1), U6.12 (B7)
- new net B_A10: J1.B30 (A10), U8.13 (B6)
- new net B_A11: J1.B31 (A11), U8.14 (B5)
- new net B_A12: J1.B33 (A12), U8.15 (B4)
- new net B_A13: J1.B34 (A13), U8.16 (B3)
- new net B_A14: J1.B37 (A14), U8.17 (B2)
- new net B_A15: J1.B38 (A15), U8.18 (B1)
- new net B_A16: J1.B41 (A16), U9.11 (B8)
- new net B_A17: J1.B42 (A17), U9.12 (B7)
- new net B_A18: J1.B45 (A18), U9.13 (B6)
- new net B_A19: J1.B46 (A19), U9.14 (B5)
- new net B_A2: J1.B17 (A2), U6.13 (B6)
- new net B_A20: J1.B49 (A20), U9.15 (B4)
- new net B_A21: J1.B50 (A21), U9.16 (B3)
- new net B_A22: J1.B51 (A22), U9.17 (B2)
- new net B_A23: J1.B54 (A23), U9.18 (B1)
- new net B_A24: J1.B55 (A24), U10.11 (B8)
- new net B_A25: J1.B58 (A25), U10.12 (B7)
- new net B_A26: J1.B59 (A26), U10.13 (B6)
- new net B_A27: J1.B62 (A27), U10.14 (B5)
- new net B_A28: J1.B63 (A28), U10.15 (B4)
- new net B_A29: J1.B66 (A29), U10.16 (B3)
- new net B_A30: J1.B67 (A30), U10.17 (B2)
- new net B_A31: J1.B70 (A31), U10.18 (B1)
- new net B_A4: J1.B19 (A4), U6.15 (B4)
- new net B_A5: J1.B20 (A5), U6.16 (B3)
- new net B_A6: J1.B23 (A6), U6.17 (B2)
- new net B_A7: J1.B24 (A7), U6.18 (B1)
- new net B_A8: J1.B27 (A8), U8.11 (B8)
- new net B_A9: J1.B28 (A9), U8.12 (B7)
- new net B_D0: J1.A72 (D0), U12.18 (B1)
- new net B_D1: J1.A69 (D1), U12.17 (B2)
- new net B_D2: J1.A68 (D2), U12.16 (B3)
- new net B_D3: J1.A65 (D3), U12.15 (B4)
- new net B_D4: J1.A64 (D4), U12.14 (B5)
- new net B_D5: J1.A61 (D5), U12.13 (B6)
- new net B_D6: J1.A60 (D6), U12.12 (B7)
- new net B_D7: J1.A57 (D7), U12.11 (B8)
- new net B_R/~{W}: J1.B77 (R/~{W}), U13.16 (B3)
- new net MAP_D10: U1.33 (D10), U5.52 (I/O)
- new net MAP_D11: U1.34 (D11), U5.54 (I/O)
- new net RECOV: J3.2 (Pin_2), U5.88 (INPUT/OE1)
- new net ~{BUSREQ}: U2.25 (~{BUSREQ}), U5.31 (I/O)
- new net ~{BUS_DMA_GNT}: U10.19 (*OE), U12.19 (*OE), U13.19 (*OE), U13.8 (A7), U5.68 (I/O), U6.19 (*OE), U8.19 (*OE), U9.19 (*OE)
- new net ~{BUS_DMA_REQ}: J1.B71 (~{DMA_REQ}), U5.69 (I/O)
- new net ~{BUS_MEM0_CS}: U13.6 (A5), U5.64 (I/O)
- new net ~{BUS_MEM1_CS}: U13.5 (A4), U5.63 (I/O)
- new net ~{BUS_MREQ}: U13.7 (A6), U5.65 (I/O)
- new net ~{B_CPU_ACK}: J1.A74 (~{CPU_ACK}), U13.18 (B1)
- new net ~{B_DMA_GNT}: J1.B72 (~{DMA_GNT}), U13.12 (B7)
- new net ~{B_MEM1_CS}: J1.B76 (~{MEM1_CS}), U13.15 (B4)
- now unconnected: U5.85 (I/O/GCLK3), U5.90 (INPUT/OE2/GCLK2)
- no-connect marks 47 -> 81
Other:
- note added: "As an option, populate J4 instead of the whole onboard programmer and use JTAG programmer."
- note added: "Device Descriptor EEPROM"
- note added: "Sense Pins Unconnected (logic 1) /DRV5v==1 --> Outputs NOT at 5V (3v3 outputs) /SENS3V == 1 --> NOT Sensitive (5v tolerant)"
- note added: "There are only 1 INT and 1 NMI on Z80, all CPU_INTX and CPU_NMI are tied to the 1 INT and 1 NMI"
- moved on the sheet: C1, C10, C11, C12, C13, C14, C15, C16, C17, C18, C2, C25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

Commit message: Added the ability to tri-state the MEM0_CS and MEM1_CS signals to allow the Dock to take over memory type selection based on addresses
Parts:
- added C31: 100n, Capacitor_SMD:C_0603_1608Metric_Pad1.08x0.95mm_HandSolder, symbol Device:C
- added U14: SN74LVC2G126DCUR, Footprints:SOP50P310X90-8N, symbol Host:SN74LVC2G126DCUR
Connections:
- net +3V3: now also C31.1, U14.8 (VCC)
- net GND: now also U13.5 (A4), U13.6 (A5), C31.2, U14.4 (GND)
- net ~{BUS_MEM0_CS}: now also U14.5 (2A); no longer U13.6 (A5)
- net ~{BUS_MEM1_CS}: now also U14.2 (1A); no longer U13.5 (A4)
- net ~{B_MEM0_CS}: now also U14.3 (2Y); no longer U13.14 (B5)
- net ~{B_MEM1_CS}: now also U14.6 (1Y); no longer U13.15 (B4)
- net ~{BUS_MEM_CS_Z}: now reaches U5.60 (I/O)
- net ~{BUS_MEM_CS_Z}: now also U14.1 (1OE), U14.7 (2OE)
- no-connect marks 81 -> 82

Commit message: Modified Pinout for easier layout Moved processing of MEM0_CS and MEM1_CS to Dock, no longer needed on Host
Parts:
- removed U14: SN74LVC2G126DCUR, Footprints:SOP50P310X90-8N, symbol Host:SN74LVC2G126DCUR
- U4: footprint SOT-23-6_MC_MCH -> Footprints:SOT-23-6_MC_MCH
Connections:
- net ~{B_MEM0_CS} is gone; now on net ~{BUS_CPU_INT}: J1.B75 (~{CPU_INT0})
- net ~{B_MEM1_CS} is gone; now on net ~{BUS_CPU_INT}: J1.B76 (~{CPU_INT1})
- net BUS_R/~{W}: now also U13.6 (A5); no longer U13.4 (A3)
- net B_R/~{W}: now also J1.A75 (R/~{W}), U13.14 (B5); no longer J1.B77 (R/~{W}), U13.16 (B3)
- net GND: now also J1.B72 (GND), U13.2 (A1), U13.3 (A2); no longer J1.A73 (GND), U13.5 (A4), U13.6 (A5)
- net ~{BUS_CPU_ACK}: now also U13.7 (A6); no longer U13.2 (A1)
- net ~{BUS_CPU_INT}: now also J1.B77 (~{CPU_INT2}), J1.B78 (~{CPU_INT3}); no longer J1.A76 (~{CPU_INT0}), J1.A77 (~{CPU_INT1}), J1.A78 (~{CPU_INT2}), J1.A79 (~{CPU_INT3})
- net ~{BUS_CPU_NMI}: now also J1.B79 (~{CPU_NMI0}), J1.B80 (~{CPU_NMI1}); no longer J1.A81 (~{CPU_NMI0}), J1.A82 (~{CPU_NMI1})
- net ~{BUS_IORQ}: now also U13.4 (A3); no longer U13.3 (A2)
- net ~{BUS_MREQ}: now also U13.5 (A4); no longer U13.7 (A6)
- net ~{BUS_READY}: now also J1.A73 (~{READY}); no longer J1.B79 (~{READY})
- net ~{BUS_RESET}: now also J1.A74 (~{RESET}); no longer J1.B73 (~{RESET})
- net ~{B_CPU_ACK}: now also J1.B74 (~{CPU_ACK}), U13.13 (B6); no longer J1.A74 (~{CPU_ACK}), U13.18 (B1)
- net ~{B_DMA_GNT}: now also J1.B73 (~{DMA_GNT}); no longer J1.B72 (~{DMA_GNT})
- net ~{B_IORQ}: now also J1.B82 (~{IORQ}), U13.16 (B3); no longer J1.B78 (~{IORQ}), U13.17 (B2)
- net ~{B_MREQ}: now also J1.B81 (~{MREQ}), U13.15 (B4); no longer J1.B74 (~{MREQ}), U13.13 (B6)
- net ~{BUS_MEM0_CS}: no longer names the net of U5.64 (I/O)
- net ~{BUS_MEM1_CS}: no longer names the net of U5.63 (I/O)
- net ~{BUS_MEM_CS_Z}: no longer names the net of U5.60 (I/O)
- no-connect marks 82 -> 87

Commit message: Removed transceivers from Z80 host with the mapper and cleaned up schematics
Parts:
- removed C19, C20, C21, C22, C23, C24, C31: 100n, Capacitor_SMD:C_0603_1608Metric_Pad1.08x0.95mm_HandSolder, symbol Device:C
- removed U10, U12, U13, U6, U8, U9: SN74LVC245ADGVR, Footprints:DGV20-M, symbol Host:SN74LVC245ADGVR
Connections:
- net B_A0 is gone; now on net A0: J1.B14 (A0)
- net B_A1 is gone; now on net A1: J1.B15 (A1)
- net B_A10 is gone; now on net A10: J1.B30 (A10)
- net B_A11 is gone; now on net A11: J1.B31 (A11)
- net B_A12 is gone; now on net A12: J1.B33 (A12)
- net B_A13 is gone; now on net A13: J1.B34 (A13)
- net B_A14 is gone; now on net A14: J1.B37 (A14)
- net B_A15 is gone; now on net A15: J1.B38 (A15)
- net B_A16 is gone; now on net A16: J1.B41 (A16)
- net B_A17 is gone; now on net A17: J1.B42 (A17)
- net B_A18 is gone; now on net A18: J1.B45 (A18)
- net B_A19 is gone; now on net A19: J1.B46 (A19)
- net B_A2 is gone; now on net A2: J1.B17 (A2)
- net B_A20 is gone; now on net A20: J1.B49 (A20)
- net B_A21 is gone; now on net A21: J1.B50 (A21)
- net B_A22 is gone; now on net A22: J1.B51 (A22)
- net B_A23 is gone; now on net A23: J1.B54 (A23)
- net B_A3 is gone; now on net A3: J1.B18 (A3)
- net B_A4 is gone; now on net A4: J1.B19 (A4)
- net B_A5 is gone; now on net A5: J1.B20 (A5)
- net B_A6 is gone; now on net A6: J1.B23 (A6)
- net B_A7 is gone; now on net A7: J1.B24 (A7)
- net B_A8 is gone; now on net A8: J1.B27 (A8)
- net B_A9 is gone; now on net A9: J1.B28 (A9)
- net B_CLK_HOST is gone; now on net CPUCLK: J1.A7 (CLK_HOST)
- net B_D0 is gone; now on net D0: J1.A72 (D0)
- net B_D1 is gone; now on net D1: J1.A69 (D1)
- net B_D2 is gone; now on net D2: J1.A68 (D2)
- net B_D3 is gone; now on net D3: J1.A65 (D3)
- net B_D4 is gone; now on net D4: J1.A64 (D4)
- net B_D5 is gone; now on net D5: J1.A61 (D5)
- net B_D6 is gone; now on net D6: J1.A60 (D6)
- net B_D7 is gone; now on net D7: J1.A57 (D7)
- net B_R/~{W} is gone; now on net BUS_R/~{W}: J1.A75 (R/~{W})
- net ~{B_CPU_ACK} is gone; now on net ~{BUS_CPU_ACK}: J1.B74 (~{CPU_ACK})
- net ~{B_DMA_GNT} is gone; now on net ~{BUS_DMA_GNT}: J1.B73 (~{DMA_GNT})
- net ~{B_IORQ} is gone; now on net ~{BUS_IORQ}: J1.B82 (~{IORQ})
- net ~{B_MREQ} is gone; now on net ~{BUS_MREQ}: J1.B81 (~{MREQ})
- net GND: now also J1.A1 (~{DRV5V}), J1.A11 (~{SENS3V})
- removed net +3V3: J1.A10 (+3V3_MAIN), J1.A9 (+3V3_MAIN), J1.B10 (+3V3_MAIN), J1.B9 (+3V3_MAIN)
- net B_A24: no longer names the net of J1.B55 (A24)
- net B_A25: no longer names the net of J1.B58 (A25)
- net B_A26: no longer names the net of J1.B59 (A26)
- net B_A27: no longer names the net of J1.B62 (A27)
- net B_A28: no longer names the net of J1.B63 (A28)
- net B_A29: no longer names the net of J1.B66 (A29)
- net B_A30: no longer names the net of J1.B67 (A30)
- net B_A31: no longer names the net of J1.B70 (A31)
- no-connect marks 87 -> 95
Other:
- note added: "Sense Pins Connected (logic 1) /VIO_5V == 1 --> Logic 5V /SLOT_PRSNT == 1 --> Always connected"
- note removed: "Sense Pins Unconnected (logic 1) /DRV5v==1 --> Outputs NOT at 5V (3v3 outputs) /SENS3V == 1 --> NOT Sensitive (5v tolerant)"
- moved on the sheet: C17, C18, C29, C30, J1A, J1C
