File: uBITz Platform Code/Host/Schem/uBITz-Host-Reference-Impl/04-Z80-Based-Host-No-Mapper/uBITz-Host-z80-Host-No-Mapper/uBITz-Host-z80-Host-No-Mapper.kicad_sch (KiCad schematic)
At the start: 24 parts, among them J3 Conn_01x02_Pin, J4 Conn_02x05_Top_Bottom, U11 24LC16BT-I_SN, U2 Z084000xP, U5 ATF1504AS-10AU100, Y1 ACH-14.31818MHZ-EK

Commit message: missing updates
Connections:
- net ~{B_IORQ} is gone; now on net ~{BUS_IORQ}: J1.B82 (~{IORQ})
- net ~{B_MREQ} is gone; now on net ~{BUS_MREQ}: J1.B81 (~{MREQ})
Changed lines of the file:
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@@
 		)
 	)
-	(label "~{B_MREQ}"
+	(label "~{BUS_MREQ}"
 		(at 657.86 386.08 0)
 		(effects
@@
 		)
 	)
-	(label "~{B_IORQ}"
+	(label "~{BUS_IORQ}"
 		(at 657.86 388.62 0)
 		(effects

Commit message: Corrected Bus width (19-bits from 20-bits) and corrected mapper wiring, which needs to be able to re-write bits A13-A15
Connections:
- net A13: no longer J1.B34 (A13)
- net A14: no longer J1.B37 (A14)
- net A15: no longer J1.B38 (A15)
- net PA13: now reaches U5.93 (I/O)
- net PA13: now also J1.B34 (A13)
- net PA14: now reaches U5.94 (I/O)
- net PA14: now also J1.B37 (A14)
- net A16 renamed PA16
- net A17 renamed PA17
- net A18 renamed PA18
- net A19: no longer names the net of J1.B46 (A19)
- net A19: no longer U5.35 (I/O)
- new net PA15: J1.B38 (A15), U5.35 (I/O)
- no-connect marks 58 -> 68
Other:
- moved on the sheet: J1A

Commit message: Removed transceivers from Z80 host with the mapper and cleaned up schematics
Other:
- note added: "Allows for JTAG Recovery Add jumper to send 12V to CPLD during programming to recover JTAG pins"
- note added: "Dual Diodes to power the CPLD only from JTAG OR from the +5V from the backplane This is to allow programming the CPLD from JTAG without powering the rest of the Host board"
- note removed: "Dual Diodes to power the CPLD only from USB OR from the +5V from the backplane This is to allow programming the CPLD from USB without powering the rest of the Host board"
Changed lines of the file:
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@@
 	(generator_version "9.0")
 	(paper "D")
+	(text "Dual Diodes to power the CPLD only\nfrom JTAG OR from the +5V from the backplane\n\nThis is to allow programming the CPLD from JTAG\nwithout powering the rest of the Host board"
+		(exclude_from_sim no)
+		(at 359.664 49.784 0)
+		(effects
+			(font
+				(size 1.27 1.27)
+			)
+			(justify left)
+		)
+	)
+	(text "Allows for JTAG Recovery\nAdd jumper to send 12V \nto CPLD during programming \nto recover JTAG pins"
+		(exclude_from_sim no)
+		(at 250.444 214.122 0)
+		(effects
+			(font
+				(size 1.27 1.27)
+			)
+			(justify left)
+		)
+	)
 	(text "There are only 1 INT and 1 NMI on Z80, \nall CPU_INTX and CPU_NMI are tied to\nthe 1 INT and 1 NMI"
 		(exclude_from_sim no)
@@
 		)
 	)
-	(text "Dual Diodes to power the CPLD only\nfrom USB OR from the +5V from the backplane\n\nThis is to allow programming the CPLD from USB\nwithout powering the rest of the Host board"
-		(exclude_from_sim no)
-		(at 355.092 50.038 0)
-		(effects
-			(font
-				(size 1.27 1.27)
-			)
-			(justify left)
-		)
-	)
 	(text "Sense Pins Connected (logic 1)\n/VIO_5V     == 1 --> Logic 5V\n/SLOT_PRSNT == 1 --> Always connected "
 		(exclude_from_sim no)
-		(at 489.204 156.464 0)
+		(at 488.188 142.494 0)
 		(effects
 			(font
@@
 	(text_box "Power and Decoupling"
 		(exclude_from_sim no)
-		(at 337.82 22.86 0)
-		(size 240.03 148.59)
+		(at 314.96 22.86 0)
+		(size 262.89 148.59)
+		(margins 0.9525 0.9525 0.9525 0.9525)
+		(stroke
+			(width 0)
+			(type solid)
+		)
+		(fill
+			(type none)
+		)
+		(effects
+			(font
+				(size 1.27 1.27)
+			)
+			(justify left top)
+		)
+	)
+	(text_box "JTAG Programming"
+		(exclude_from_sim no)
+		(at 236.22 203.2 0)
+		(size 57.15 91.44)
+		(margins 0.9525 0.9525 0.9525 0.9525)
+		(stroke
+			(width 0)
+			(type solid)
+		)
+		(fill
+			(type none)
+		)
+		(effects
+			(font
+				(size 1.27 1.27)
+			)
+			(justify left top)
+		)
+	)
+	(text_box "MMU and uBITz bus adaptor"
+		(exclude_from_sim no)
+		(at 21.59 179.07 0)
+		(size 283.21 201.93)
+		(margins 0.9525 0.9525 0.9525 0.9525)
+		(stroke
+			(width 0)
+			(type solid)
+		)
+		(fill
+			(type none)
+		)
+		(effects
+			(font
+				(size 1.27 1.27)
+			)
+			(justify left top)
+		)
+	)
+	(text_box "Edge Connector"
+		(exclude_from_sim no)
+		(at 314.96 179.07 0)
+		(size 262.89 201.93)
 		(margins 0.9525 0.9525 0.9525 0.9525)
 		(stroke
@@
 		(exclude_from_sim no)
 		(at 21.59 22.86 0)
-		(size 288.29 148.59)
+		(size 283.21 148.59)
 		(margins 0.9525 0.9525 0.9525 0.9525)
 		(stroke
@@
 		)
 	)
-	(text_box "uBITz Dock Connector"
-		(exclude_from_sim no)
-		(at 881.38 603.25 0)
-		(size 223.52 160.02)
-		(margins 0.9525 0.9525 0.9525 0.9525)
-		(stroke
-			(width 0)
-			(type solid)
-		)
-		(fill
-			(type none)
-		)
-		(effects
-			(font
-				(size 1.27 1.27)
-			)
-			(justify right top)
-		)
-	)
